File: hardware/hardware/hardware.kicad_sch (KiCad schematic)
At the start: 18 parts, among them U1 STM32L432KCUx

Commit message: led matrix kicad
Parts:
- added D100, D101, D102, D103, D104, D105, D106, D107, D108, D109, D110, D111, D112, D114, D115, D116, D117, D118, D119, D120, D123, D124, D125, D126, D127, D128, D132, D133, D134, D135, D136, D141, D142, D143, D144, D145, D146, D147, D148, D153, D154, D155, D156, D157, D161, D162, D163, D164, D165, D166, D169, D17, D170, D171, D172, D173, D174, D175, D177, D178, D179, D18, D180, D181, D182, D183, D185, D186, D187, D188, D189, D19, D190, D191, D193, D194, D195, D196, D197, D198, D199, D20, D201, D202, D203, D204, D205, D206, D207, D209, D21, D210, D211, D212, D213, D214, D215, D217, D218, D219, D22, D220, D221, D222, D223, D225, D226, D227, D228, D229, D23, D230, D231, D233, D234, D235, D236, D237, D238, D239, D24, D241, D242, D243, D244, D245, D246, D247, D249, D25, D250, D251, D252, D253, D254, D257, D258, D259, D260, D261, D265, D266, D267, D268, D28, D29, D30, D31, D32, D33, D34, D35, D36, D37, D38, D39, D40, D41, D42, D43, D44, D45, D46, D47, D48, D49, D50, D51, D52, D53, D54, D55, D56, D57, D58, D59, D60, D61, D62, D63, D64, D65, D66, D67, D68, D69, D70, D71, D72, D73, D74, D75, D76, D77, D78, D79, D80, D81, D82, D83, D84, D85, D86, D87, D88, D89, D90, D91, D92, D93, D94, D95, D96, D97, D98, D99: LED, symbol Device:LED
Connections:
- new net: D100.2 (A), D101.1 (K), D107.2 (A), D108.1 (K), D114.2 (A), D115.1 (K), D157.2 (A), D164.2 (A), D165.1 (K), D171.2 (A), D172.1 (K), D178.2 (A), D179.1 (K), D185.2 (A), D186.1 (K), D193.1 (K), D76.2 (A), D79.2 (A), D80.1 (K), D86.2 (A), D87.1 (K), D93.2 (A), D94.1 (K)
- new net: D100.1 (K), D108.2 (A), D109.1 (K), D117.2 (A), D118.1 (K), D126.2 (A), D127.1 (K), D135.2 (A), D136.1 (K), D144.2 (A), D265.2 (A), D30.2 (A), D31.2 (A), D32.1 (K), D33.1 (K), D41.1 (K), D43.1 (K), D46.2 (A), D47.2 (A), D48.1 (K), D53.2 (A), D54.1 (K), D57.1 (K), D81.2 (A), D82.1 (K), D90.2 (A), D91.1 (K), D99.2 (A)
- new net: D101.2 (A), D102.1 (K), D110.2 (A), D111.1 (K), D119.2 (A), D120.1 (K), D128.2 (A), D24.1 (K), D249.1 (K), D257.2 (A), D258.1 (K), D266.2 (A), D267.2 (A), D28.1 (K), D29.1 (K), D39.1 (K), D41.2 (A), D42.1 (K), D44.2 (A), D45.1 (K), D47.1 (K), D83.2 (A), D84.1 (K), D92.2 (A), D93.1 (K)
- new net: D105.2 (A), D106.1 (K), D155.2 (A), D156.1 (K), D162.2 (A), D163.1 (K), D169.2 (A), D170.1 (K), D177.1 (K), D68.2 (A), D71.2 (A), D72.1 (K), D74.2 (A), D75.1 (K), D77.2 (A), D78.1 (K), D84.2 (A), D85.1 (K), D91.2 (A), D92.1 (K), D98.2 (A), D99.1 (K)
- new net: D106.2 (A), D107.1 (K), D115.2 (A), D116.1 (K), D124.2 (A), D125.1 (K), D133.2 (A), D134.1 (K), D142.2 (A), D143.2 (A), D34.2 (A), D35.2 (A), D36.1 (K), D37.1 (K), D42.2 (A), D43.2 (A), D44.1 (K), D55.2 (A), D56.1 (K), D58.2 (A), D59.1 (K), D61.2 (A), D62.1 (K), D65.1 (K), D81.1 (K), D89.1 (K), D97.2 (A), D98.1 (K)
- new net D1: D217.1 (K), D22.1 (K), D225.2 (A), D226.1 (K), D23.2 (A), D234.2 (A), D235.1 (K), D243.2 (A), D244.1 (K), D252.2 (A), D253.1 (K), D261.2 (A), D28.2 (A), D31.1 (K), D33.2 (A), D34.1 (K), D36.2 (A), D69.1 (K), D73.2 (A), D74.1 (K), D78.2 (A), D79.1 (K), D87.2 (A), D88.1 (K), D96.2 (A)
- new net D10: D136.2 (A), D143.1 (K), D144.1 (K), D145.2 (A), D146.1 (K), D154.2 (A), D155.1 (K), D163.2 (A), D164.1 (K), D172.2 (A), D173.1 (K), D181.2 (A), D182.1 (K), D190.2 (A), D191.1 (K), D199.2 (A), D207.2 (A), D214.2 (A), D215.1 (K), D221.2 (A), D222.1 (K), D228.2 (A), D229.1 (K), D235.2 (A), D236.1 (K), D242.2 (A), D243.1 (K), D249.2 (A), D250.1 (K), D257.1 (K)
- new net D11: D105.1 (K), D114.1 (K), D123.1 (K), D132.1 (K), D141.2 (A), D146.2 (A), D147.1 (K), D153.2 (A), D154.1 (K), D161.1 (K), D38.2 (A), D39.2 (A), D40.1 (K), D60.2 (A), D63.2 (A), D64.1 (K), D66.2 (A), D67.1 (K), D69.2 (A), D70.1 (K), D73.1 (K), D82.2 (A), D83.1 (K), D89.2 (A), D90.1 (K), D97.1 (K)
- new net D12: D120.2 (A), D127.2 (A), D128.1 (K), D134.2 (A), D135.1 (K), D141.1 (K), D142.1 (K), D147.2 (A), D148.1 (K), D156.2 (A), D157.1 (K), D165.2 (A), D166.1 (K), D174.2 (A), D175.1 (K), D183.2 (A), D191.2 (A), D198.2 (A), D199.1 (K), D205.2 (A), D206.1 (K), D212.2 (A), D213.1 (K), D219.2 (A), D220.1 (K), D226.2 (A), D227.1 (K), D233.2 (A), D234.1 (K), D241.1 (K)
- new net D13: D148.2 (A)
- new net D14: D104.2 (A), D111.2 (A), D112.1 (K), D118.2 (A), D119.1 (K), D125.2 (A), D126.1 (K), D132.2 (A), D133.1 (K), D17.2 (A), D175.2 (A), D18.1 (K), D182.2 (A), D183.1 (K), D189.2 (A), D19.2 (A), D190.1 (K), D196.2 (A), D197.1 (K), D20.1 (K), D203.2 (A), D204.1 (K), D210.2 (A), D211.1 (K), D217.2 (A), D218.1 (K), D225.1 (K)
- new net D15: D18.2 (A)
- new net D16: D102.2 (A), D103.1 (K), D109.2 (A), D110.1 (K), D116.2 (A), D117.1 (K), D123.2 (A), D124.1 (K), D166.2 (A), D17.1 (K), D173.2 (A), D174.1 (K), D180.2 (A), D181.1 (K), D187.2 (A), D188.1 (K), D194.2 (A), D195.1 (K), D20.2 (A), D201.2 (A), D202.1 (K), D209.1 (K), D88.2 (A), D95.2 (A), D96.1 (K)
- new net D2: D201.1 (K), D209.2 (A), D21.1 (K), D210.1 (K), D218.2 (A), D219.1 (K), D227.2 (A), D228.1 (K), D236.2 (A), D237.1 (K), D245.2 (A), D246.1 (K), D25.2 (A), D254.2 (A), D29.2 (A), D30.1 (K), D32.2 (A), D61.1 (K), D65.2 (A), D66.1 (K), D70.2 (A), D71.1 (K), D75.2 (A), D76.1 (K), D80.2 (A)
- new net D3: D103.2 (A), D104.1 (K), D112.2 (A), D233.1 (K), D241.2 (A), D242.1 (K), D250.2 (A), D251.1 (K), D259.2 (A), D260.1 (K), D268.2 (A), D35.1 (K), D37.2 (A), D38.1 (K), D40.2 (A), D45.2 (A), D46.1 (K), D48.2 (A), D77.1 (K), D85.2 (A), D86.1 (K), D94.2 (A), D95.1 (K)
- new net D4: D185.1 (K), D193.2 (A), D194.1 (K), D202.2 (A), D203.1 (K), D21.2 (A), D211.2 (A), D212.1 (K), D22.2 (A), D220.2 (A), D221.1 (K), D229.2 (A), D23.1 (K), D230.1 (K), D238.2 (A), D239.1 (K), D24.2 (A), D247.2 (A), D25.1 (K), D53.1 (K), D57.2 (A), D58.1 (K), D62.2 (A), D63.1 (K), D67.2 (A), D68.1 (K), D72.2 (A)
- new net D5: D49.1 (K)
- new net D6: D169.1 (K), D177.2 (A), D178.1 (K), D186.2 (A), D187.1 (K), D195.2 (A), D196.1 (K), D204.2 (A), D205.1 (K), D213.2 (A), D214.1 (K), D222.2 (A), D223.1 (K), D231.2 (A), D239.2 (A), D246.2 (A), D247.1 (K), D253.2 (A), D254.1 (K), D260.2 (A), D261.1 (K), D267.1 (K), D268.1 (K), D49.2 (A), D50.1 (K), D54.2 (A), D55.1 (K), D59.2 (A), D60.1 (K), D64.2 (A)
- new net D7: D50.2 (A), D51.1 (K)
- new net D8: D153.1 (K), D161.2 (A), D162.1 (K), D170.2 (A), D171.1 (K), D179.2 (A), D180.1 (K), D188.2 (A), D189.1 (K), D197.2 (A), D198.1 (K), D206.2 (A), D207.1 (K), D223.2 (A), D230.2 (A), D231.1 (K), D237.2 (A), D238.1 (K), D244.2 (A), D245.1 (K), D251.2 (A), D252.1 (K), D258.2 (A), D259.1 (K), D265.1 (K), D266.1 (K), D51.2 (A), D52.1 (K), D56.2 (A)
- new net D9: D145.1 (K), D52.2 (A)
Other:
- moved on the sheet: D1, D10, D11, D12, D13, D14, D15, D16, D2, D3, D4, D5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
